File: Hardware/Qwiic GPS-RTK2 - ublox ZED-F9P.brd (EAGLE design)
At the start: 43.2 x 43.2 mm, 136 parts, among them J1 Radio, J13 U.FL, J3 PTH, U2 3.3V, U3 ZED-F9P

Commit message: Adds reflowable battery and uses all parts from SparkFun Libraries
Parts:
- removed B1: 6.8MM_COIN_CELL, SparkFun-Batteries:BATTCON-6.8MM
- removed J3: PTH, SparkX:1X04_NO_SILK
- added BT1: ML414H_IV01E_BATTERY, SparkFun-Batteries:ML414H_IV01E
- added J8: (no value), SparkFun-Connectors:1X04_NO_SILK
- J2, J4: value (none) -> Qwiic Right Angle; device SparkFun-Connectors:1X04_1MM_RA -> SparkFun-Connectors:JST04_1MM_RA
- JP1, JP2, JP3: value (none) -> JUMPER-SMT_2_NC_TRACE_SILK
- JP101, JP31, JP41, JP91: value STAND-OFF -> STAND-OFFTIGHT; device SparkFun:STAND-OFF -> SparkFun-Hardware:STAND-OFF-TIGHT
- JP21, JP61, JP71, JP81: device SparkFun:MICRO-FIDUCIAL -> SparkFun-Aesthetics:FIDUCIAL-MICRO
- JP4: value (none) -> JUMPER-SMT_2_NO_SILK
- JP5: value (none) -> JUMPER-SMT_3_2-NC_TRACE_SILK
- U3: device ZED-F9P:ZED-F9P -> SparkFun-GPS:ZED-F9P
Connections:
- net 3.3V: now also J8.2; no longer J3.2
- net BACKUP: now also BT1.+; no longer B1.+
- net GND: now also BT1.-, J8.1; no longer B1.-, J3.1
- net SCL/SCK: now also J8.4; no longer J3.4
- net SDA/!CS: now also J8.3; no longer J3.3
Routing:
- net BACKUP: track 20.9 -> 21.6 mm
- net UNP_D-: track 6.29 -> 6.97 mm
- net 5V: track 52.8 -> 53.5 mm
- net GND: vias 174 -> 175
Other:
- board text added: "+"
- board text added: "-"
- board text added: "Nathan Seidle"
- board text added: "Revised By: Elias Santistevan"
- board text added: "v20"
- board text removed: "v11"

Commit message: Adds panel for v20
Changed lines of the file:
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@@
 <layer number="20" name="Dimension" color="15" fill="1" visible="yes" active="yes"/>
 <layer number="21" name="tPlace" color="16" fill="1" visible="yes" active="yes"/>
-<layer number="22" name="bPlace" color="14" fill="1" visible="no" active="yes"/>
+<layer number="22" name="bPlace" color="14" fill="1" visible="yes" active="yes"/>
 <layer number="23" name="tOrigins" color="15" fill="1" visible="yes" active="yes"/>
 <layer number="24" name="bOrigins" color="15" fill="1" visible="yes" active="yes"/>
@@
 <layer number="115" name="ReferenceISLANDS" color="7" fill="1" visible="no" active="no"/>
 <layer number="116" name="Patch_BOT" color="9" fill="4" visible="no" active="no"/>
-<layer number="117" name="PM_Ref" color="26" fill="1" visible="yes" active="yes"/>
+<layer number="117" name="PM_Ref" color="26" fill="1" visible="no" active="yes"/>
 <layer number="118" name="Rect_Pads" color="7" fill="1" visible="no" active="no"/>
-<layer number="119" name="PF_Ref" color="31" fill="1" visible="yes" active="yes"/>
-<layer number="120" name="WFL_Ref" color="25" fill="1" visible="yes" active="yes"/>
+<layer number="119" name="PF_Ref" color="31" fill="1" visible="no" active="yes"/>
+<layer number="120" name="WFL_Ref" color="25" fill="1" visible="no" active="yes"/>
 <layer number="121" name="_tsilk" color="7" fill="1" visible="no" active="no"/>
 <layer number="122" name="_bsilk" color="7" fill="1" visible="no" active="no"/>
@@
 <via x="16.7132" y="19.939" extent="1-16" drill="0.3048"/>
 <via x="11.938" y="18.415" extent="1-16" drill="0.3048"/>
-<wire x1="7.62" y1="25.609340625" x2="7.62" y2="25.4" width="0.1524" layer="1"/>
 <via x="7.62" y="25.4" extent="1-16" drill="0.3048"/>
 <wire x1="16.7132" y1="19.939" x2="11.938" y2="19.939" width="0.1524" layer="16"/>
@@
 <contactref element="J5" pad="SHLD2"/>
 <contactref element="J5" pad="SHLD3"/>
-<polygon width="0.1524" layer="1">
+<polygon width="0.1524" layer="1" thermals="no">
 <vertex x="0" y="17.272"/>
 <vertex x="5.842" y="17.272"/>
@@
 <vertex x="0" y="7.874"/>
 </polygon>
-<wire x1="5.435" y1="17.02" x2="5.435" y2="17.02" width="0" layer="19" extent="1-16"/>
-<wire x1="5.435" y1="8.38" x2="5.435" y2="8.38" width="0" layer="19" extent="1-16"/>
-<wire x1="1.255" y1="8.38" x2="1.255" y2="8.38" width="0" layer="19" extent="1-16"/>
+<via x="3.048" y="12.7" extent="1-16" drill="0.3048"/>
+<via x="4.445" y="9.1948" extent="1-16" drill="0.3048"/>
+<via x="4.826" y="14.478" extent="1-16" drill="0.3048"/>
 </signal>
 <signal name="GPS_ANT1">
@@
 <contactref element="R16" pad="2"/>
 <contactref element="J5" pad="B5"/>
-<wire x1="6.01" y1="10.95" x2="4.6" y2="10.95" width="0.1524" layer="1"/>
-<wire x1="4.025" y1="10.375" x2="4.025" y2="6.985" width="0.1524" layer="1"/>
-<wire x1="4.6" y1="10.95" x2="4.025" y2="10.375" width="0.1524" layer="1"/>
+<wire x1="6.01" y1="10.95" x2="4.3968" y2="10.95" width="0.1524" layer="1"/>
+<wire x1="3.898" y1="10.4512" x2="3.898" y2="7.112" width="0.1524" layer="1"/>
+<wire x1="3.898" y1="7.112" x2="4.025" y2="6.985" width="0.1524" layer="1"/>
+<wire x1="4.3968" y1="10.95" x2="3.898" y2="10.4512" width="0.1524" layer="1"/>
 </signal>
 <signal name="UNP_D+">
